Commit message: 机械臂解决了几个小问题,但面临仿真启动后rviz2机械臂会莫名转动,mujoco机械臂无相应的大问题

File: src/arm/model/arm.urdf (robot description, URDF)
Before this commit: robot arm, 6 links, 5 joints
Joints:
- joint joint2: origin xyz=0.3275 -0.0335 0.0485 rpy=1.5708 0 0 -> xyz=0.3275 -0.0335 0.0485 rpy=1.5708 -1.5708 0
- joint joint3: origin xyz=0.3695 0 -0.044 rpy=0 0 0 -> xyz=0.3695 0 -0.044 rpy=0 0 -1.5708

Commit message: 修改了转动角度正负问题

File: src/arm/model/arm.urdf (robot description, URDF)
Before this commit: robot arm, 6 links, 5 joints
Joints:
- joint joint2: axis 0 0 1 -> 0 0 -1; origin xyz=0.3275 -0.0335 0.0485 rpy=1.5708 -1.5708 0 -> xyz=0.3275 -0.0335 0.0485 rpy=1.5708 3.1416 0
- joint joint4: axis 0 0 1 -> 0 0 -1; origin xyz=0.2 0.004 -0.026 rpy=0 0 0 -> xyz=0.2 0.004 -0.026 rpy=0 0 1.5708

Commit message: 已经调好的机械臂代码

File: src/arm/model/arm.urdf (robot description, URDF)
Before this commit: robot arm, 6 links, 5 joints
Joints:
- joint joint1: axis 0 0 -1 -> 0 0 1
- joint joint3: limit lower=-3.1416 upper=3.1416 effort=0 velocity=0 -> lower=0 upper=1.5708 effort=0 velocity=0
