Commit message: 可以控制末端俯仰了

File: src/arm/model/armarm.urdf (robot description, URDF)
Before this commit: robot arm, 6 links, 5 joints
Links:
- removed link world
- added link link5, mass 6.72485772348953; collision box size=0.001 0.001 0.001; visual box size=0.001 0.001 0.001
- link link2: mass 0.549716905790998 -> 0.425516880933423
Joints:
- removed joint world_joint
- added joint joint5: type fixed, parent link4, child link5, origin xyz=-0.033 -0.0904 0.02425 rpy=1.5708 0 0, axis 0 0 0
- joint joint2: limit lower=-3.1416 upper=3.1416 effort=0 velocity=0 -> lower=-3.14159 upper=3.14159 effort=0 velocity=0; origin xyz=0.3275 -0.0335 0.0485 rpy=1.5708 3.1416 0 -> xyz=0.32753 -0.04351 0.0325 rpy=1.5708 3.1416 0
- joint joint3: limit lower=0 upper=1.5708 effort=0 velocity=0 -> lower=-3.14159 upper=3.14159 effort=0 velocity=0; origin xyz=0.3695 0 -0.044 rpy=0 0 -1.5708 -> xyz=0.34 0 -0.0435 rpy=0 0 -1.5708
- joint joint4: limit lower=-3.1416 upper=3.1416 effort=0 velocity=0 -> lower=-3.14159 upper=3.14159 effort=0 velocity=0; origin xyz=0.2 0.004 -0.026 rpy=0 0 1.5708 -> xyz=0.17 -0.020156 -0.02375 rpy=0 0 1.5708

Commit message: 完成对末端的控制

File: src/arm/model/armarm.urdf (robot description, URDF)
Before this commit: robot armarm, 6 links, 5 joints
Joints:
- joint joint5: origin xyz=-0.033 -0.0904 0.02425 rpy=1.5708 0 0 -> xyz=-0.033 -0.0904 0.02425 rpy=-1.5708 0 3.14159
